Commit message: Adjusting URDF Values

File: urdf/rover.urdf.xacro (robot description, xacro)
@@ -4,7 +4,8 @@
   <material name="black"><color rgba="0.06 0.06 0.06 1.0"/></material>
   <material name="tread"><color rgba="0.22 0.22 0.22 1.0"/></material>
+  <material name="yellow"><color rgba="1.0 0.9 0.0 1.0"/></material>
   <!-- Tune these to change tread appearance across all wheels -->
-  <xacro:property name="wheel_radius"   value="0.080"/>
-  <xacro:property name="wheel_length"   value="0.070"/>
+  <xacro:property name="wheel_radius"   value="0.0762"/>
+  <xacro:property name="wheel_length"   value="0.04445"/>
   <xacro:property name="tread_diameter" value="0.012"/> <!-- groove depth in diameter units; inner_r = wheel_radius - tread_diameter/2 -->
   <xacro:property name="tread_count"    value="8"/>
@@ -17,6 +18,8 @@
   <xacro:property name="tread_block_l" value="${wheel_length - 0.015}"/>
   <link name="base_link">
-    <visual><geometry><box size="0.35 0.28 0.05"/></geometry><origin xyz="0 0 -0.025"/><material name="gray"/></visual>
-    <collision><geometry><box size="0.35 0.28 0.05"/></geometry></collision>
+    <visual><geometry><box size="0.254 0.2159 0.05"/></geometry><origin xyz="0 0 -0.025"/><material name="gray"/></visual>
+    <visual><geometry><box size="0.127 0.0762 0.1016"/></geometry><origin xyz="-0.0635 0 0.0508"/><material name="yellow"/></visual>
+    <collision><geometry><box size="0.254 0.2159 0.05"/></geometry></collision>
+    <collision><geometry><box size="0.127 0.0762 0.1016"/></geometry><origin xyz="-0.0635 0 0.0508"/></collision>
     <inertial><mass value="2.7"/><inertia ixx="0.02" ixy="0" ixz="0" iyy="0.02" iyz="0" izz="0.02"/></inertial>
   </link>
@@ -53,7 +56,7 @@
     </joint>
   </xacro:macro>
-  <xacro:wheel name="front_left"  x=" 0.125" y=" 0.16"/>
-  <xacro:wheel name="front_right" x=" 0.125" y="-0.16"/>
-  <xacro:wheel name="rear_left"   x="-0.125" y=" 0.16"/>
-  <xacro:wheel name="rear_right"  x="-0.125" y="-0.16"/>
+  <xacro:wheel name="front_left"  x=" 0.1016" y=" 0.13335"/>
+  <xacro:wheel name="front_right" x=" 0.1016" y="-0.13335"/>
+  <xacro:wheel name="rear_left"   x="-0.1016" y=" 0.13335"/>
+  <xacro:wheel name="rear_right"  x="-0.1016" y="-0.13335"/>
 </robot>

Commit message: Lidar producing data

File: urdf/rover.urdf.xacro (robot description, xacro)
@@ -60,3 +60,17 @@
   <xacro:wheel name="rear_left"   x="-0.1016" y=" 0.13335"/>
   <xacro:wheel name="rear_right"  x="-0.1016" y="-0.13335"/>
+  <!-- RPLIDAR A2M12 — mounted in front of the yellow electronics box -->
+  <link name="laser">
+    <visual>
+      <geometry><cylinder radius="0.0351" length="0.0407"/></geometry>
+      <material name="lidar_blue"><color rgba="0.1 0.4 0.8 1.0"/></material>
+    </visual>
+    <collision><geometry><cylinder radius="0.0351" length="0.0407"/></geometry></collision>
+    <inertial><mass value="0.17"/><inertia ixx="0.0001" ixy="0" ixz="0" iyy="0.0001" iyz="0" izz="0.0001"/></inertial>
+  </link>
+  <joint name="laser_joint" type="fixed">
+    <parent link="base_link"/>
+    <child link="laser"/>
+    <origin xyz="0.08 0.0 0.236" rpy="0 0 ${pi}"/>
+  </joint>
 </robot>

Commit message: adjusting mesh size

File: urdf/rover.urdf.xacro (robot description, xacro)
@@ -63,8 +63,8 @@
   <link name="laser">
     <visual>
-      <geometry><cylinder radius="0.0351" length="0.0407"/></geometry>
+      <geometry><cylinder radius="0.0381" length="0.04445"/></geometry>
       <material name="lidar_blue"><color rgba="0.1 0.4 0.8 1.0"/></material>
     </visual>
-    <collision><geometry><cylinder radius="0.0351" length="0.0407"/></geometry></collision>
+    <collision><geometry><cylinder radius="0.0381" length="0.04445"/></geometry></collision>
     <inertial><mass value="0.17"/><inertia ixx="0.0001" ixy="0" ixz="0" iyy="0.0001" iyz="0" izz="0.0001"/></inertial>
   </link>
@@ -72,5 +72,5 @@
     <parent link="base_link"/>
     <child link="laser"/>
-    <origin xyz="0.08 0.0 0.236" rpy="0 0 ${pi}"/>
+    <origin xyz="0.0508 0.0 0.238" rpy="0 0 ${pi}"/>
   </joint>
 </robot>

Commit message: Lidar mapping working

File: urdf/rover.urdf.xacro (robot description, xacro)
@@ -17,4 +17,13 @@
   <xacro:property name="tread_block_w" value="${2.0 * pi * tread_block_r / tread_count - tread_gap}"/>
   <xacro:property name="tread_block_l" value="${wheel_length - 0.015}"/>
+  <!-- Ground-projection frame: sits on the floor directly under base_link so the
+       2D map/odom plane lands at the floor instead of through the chassis.
+       0.1012 = wheel_joint z (0.025) + wheel_radius (0.0762). -->
+  <link name="base_footprint"/>
+  <joint name="base_footprint_joint" type="fixed">
+    <parent link="base_footprint"/>
+    <child link="base_link"/>
+    <origin xyz="0 0 0.1012" rpy="0 0 0"/>
+  </joint>
   <link name="base_link">
     <visual><geometry><box size="0.254 0.2159 0.05"/></geometry><origin xyz="0 0 -0.025"/><material name="gray"/></visual>

Commit message: working depth camera data

File: urdf/rover.urdf.xacro (robot description, xacro)
@@ -70,10 +70,14 @@
   <xacro:wheel name="rear_right"  x="-0.1016" y="-0.13335"/>
   <!-- RPLIDAR A2M12 — mounted in front of the yellow electronics box -->
+  <xacro:property name="lidar_radius" value="0.0381"/>
+  <xacro:property name="lidar_length" value="0.04445"/>
+  <xacro:property name="lidar_x"      value="0.0508"/>  <!-- 2" forward of base_link -->
+  <xacro:property name="lidar_z"      value="0.127"/>   <!-- 5" up from base_link -->
   <link name="laser">
     <visual>
-      <geometry><cylinder radius="0.0381" length="0.04445"/></geometry>
+      <geometry><cylinder radius="${lidar_radius}" length="${lidar_length}"/></geometry>
       <material name="lidar_blue"><color rgba="0.1 0.4 0.8 1.0"/></material>
     </visual>
-    <collision><geometry><cylinder radius="0.0381" length="0.04445"/></geometry></collision>
+    <collision><geometry><cylinder radius="${lidar_radius}" length="${lidar_length}"/></geometry></collision>
     <inertial><mass value="0.17"/><inertia ixx="0.0001" ixy="0" ixz="0" iyy="0.0001" iyz="0" izz="0.0001"/></inertial>
   </link>
@@ -81,5 +85,30 @@
     <parent link="base_link"/>
     <child link="laser"/>
-    <origin xyz="0.0508 0.0 0.238" rpy="0 0 ${pi}"/>
+    <origin xyz="${lidar_x} 0.0 ${lidar_z}" rpy="0 0 ${pi}"/>
   </joint>
+  <!-- Intel RealSense D455 — rough model (~124 x 26 x 29 mm, W x H x D): grey
+       bar body + black glass front. This link IS camera_link (the realsense
+       root frame, +x forward), so the driver's optical frames hang off it. -->
+  <xacro:macro name="d455_camera" params="name parent xyz rpy">
+    <link name="${name}">
+      <visual> <!-- grey body -->
+        <geometry><box size="0.029 0.124 0.026"/></geometry>
+        <material name="gray"/>
+      </visual>
+      <visual> <!-- black glass front (lens window) -->
+        <origin xyz="0.0145 0 0"/>
+        <geometry><box size="0.004 0.108 0.020"/></geometry>
+        <material name="black"/>
+      </visual>
+      <inertial><mass value="0.072"/><inertia ixx="0.0001" ixy="0" ixz="0" iyy="0.0001" iyz="0" izz="0.0001"/></inertial>
+    </link>
+    <joint name="${name}_joint" type="fixed">
+      <parent link="${parent}"/>
+      <child link="${name}"/>
+      <origin xyz="${xyz}" rpy="${rpy}"/>
+    </joint>
+  </xacro:macro>
+  <!-- 5" forward, 3.25" up from base_link -->
+  <xacro:d455_camera name="camera_link" parent="base_link" rpy="0 0 0"
+      xyz="0.127 0 0.08255"/>
 </robot>
